File: hardware/legofruit/legofruitv2/legofruitv2.kicad_sch (KiCad schematic)
At the start: 44 parts, among them J1 Conn_01x06, J10 SERVO4, J11 Conn_01x03, J12 MOTOR1, J2 USB_B_Micro, J3 Conn_ARM_JTAG_SWD_10, J4 MOTOR2, J5 SERVO1, J6 SERVO2, J7 SERVO3, J8 UART, J9 POWER, Q1 DMG2305, U1 MDBT50Q-1MV2, U2 MOTOR2_DRV, U4 AP2112K-3.3, U5 MOTOR1_DRV, Y1 32768 KHz

Commit message: Device driver version
Parts:
- removed BT1: Battery, Battery:BatteryHolder_Keystone_2479_3xAAA, symbol Device:Battery
- removed J8: UART, Connector_PinHeader_2.54mm:PinHeader_1x02_P2.54mm_Vertical, symbol Connector_Generic:Conn_01x02
- added J13: GPIO, Connector_PinHeader_2.54mm:PinHeader_1x08_P2.54mm_Vertical, symbol Connector_Generic:Conn_01x08
Connections:
- net +3.3V: now also J13.8 (Pin_8)
- net GND: now also J13.7 (Pin_7)
- net at U1.50 (P1.02): now also J13.5 (Pin_5)
- net at U1.56 (P1.04): now also J13.3 (Pin_3)
- net at U1.57 (P1.06): now also J13.1 (Pin_1)
- net at U1.59 (P1.05): now also J13.2 (Pin_2)
- net at U1.60 (P1.03): now also J13.4 (Pin_4)
- net at U1.61 (P1.01): now also J13.6 (Pin_6)
- no-connect marks 25 -> 21
Other:
- note added: "I2c"
